File: pcb/BleShield.brd (EAGLE design)
At the start: 53.3 x 48.3 mm, 30 parts, among them Q1 32.768K, 10ppm, SW1 SPST_TACT-EVQQ2, SW2 SPST_TACT-EVQQ2, U1 ARDUINO_SHIELDNOHOLES

Commit message: Put the 47k resistors in for the pick&place machine
Parts:
- R12, R13: value DNP -> 47k
Changed lines of the file:
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@@
 <attribute name="VALUE" x="7.484" y="39.103" size="0.4064" layer="27"/>
 </element>
-<element name="R12" library="SparkFun" package="0805" value="DNP" x="8.5" y="37.5" smashed="yes">
+<element name="R12" library="SparkFun" package="0805" value="47k" x="8.5" y="37.5" smashed="yes">
 <attribute name="VALUE" x="7.484" y="36.103" size="0.4064" layer="27"/>
 </element>
-<element name="R13" library="SparkFun" package="0805" value="DNP" x="8.5" y="36" smashed="yes">
+<element name="R13" library="SparkFun" package="0805" value="47k" x="8.5" y="36" smashed="yes">
 <attribute name="VALUE" x="7.484" y="34.603" size="0.4064" layer="27"/>
 </element>
